Commit message: now drok3 can climb stairs

File: urdf/drok3_description2.urdf (robot description, URDF)
Before this commit: robot drok3_description2, 26 links, 24 joints
Links:
- added link l11_link, mass 0.697502716828587; collision mesh filename=package://drok3_description2/meshes/L1_link.STL; visual mesh filename=package://drok3_description2/meshes/L1_link.STL
- added link l12_link, mass 0.697502716828589; collision mesh filename=package://drok3_description2/meshes/L2_link.STL; visual mesh filename=package://drok3_description2/meshes/L2_link.STL
- added link r11_link, mass 0.697502716828587; collision mesh filename=package://drok3_description2/meshes/R1_link.STL; visual mesh filename=package://drok3_description2/meshes/R1_link.STL
- added link r12_link, mass 0.697502716828588; collision mesh filename=package://drok3_description2/meshes/R2_link.STL; visual mesh filename=package://drok3_description2/meshes/R2_link.STL
Joints:
- added joint l11_link_joint: type continuous, parent base_link, child l11_link, origin xyz=-0.22424 0.25972 -0.028 rpy=0 0 0, axis 0 1 0
- added joint l12_link_joint: type continuous, parent base_link, child l12_link, origin xyz=0.22576 0.25972 -0.028 rpy=0 0 0, axis 0 1 0
- added joint r10_link_joint: type continuous, parent base_link, child r10_link, origin xyz=0.07576 -0.25972 -0.028 rpy=0 0 0, axis 0 1 0
- added joint r11_link_joint: type continuous, parent base_link, child r11_link, origin xyz=-0.22424 -0.25972 -0.028 rpy=0 0 0, axis 0 1 0
- added joint r12_link_joint: type continuous, parent base_link, child r12_link, origin xyz=0.22576 -0.25972 -0.028 rpy=0 0 0, axis 0 1 0
- joint r2_link_joint: origin xyz=0.07576 -0.25972 -0.028 rpy=0 0 0 -> xyz=0.12576 -0.25972 -0.028 rpy=0 0 0

Commit message: first commit 2021-03-29

File: urdf/drok3_description2.urdf (robot description, URDF)
Before this commit: robot drok3_description2, 30 links, 29 joints
Links:
- link l11_link: geometry collision mesh filename=package://drok3_description2/meshes/L1_link.STL
- link l12_link: geometry collision mesh filename=package://drok3_description2/meshes/L2_link.STL
- link r11_link: geometry collision mesh filename=package://drok3_description2/meshes/R1_link.STL
- link r12_link: geometry collision mesh filename=package://drok3_description2/meshes/R2_link.STL

Commit message: add lidar, add parking world, modify friction 2021-03-31

File: urdf/drok3_description2.urdf (robot description, URDF)
Before this commit: robot drok3_description2, 30 links, 29 joints
Links:
- added link lidar_link, mass 0.5
Joints:
- added joint lidar_joint: type fixed, parent base_link, child lidar_link, origin xyz=0.5 -0.000335907486689213 0.0569327313017182 rpy=0 0 0, axis 0 1 0

Commit message: remove base_footprint_link 2021-05-25

File: urdf/drok3_description2.urdf (robot description, URDF)
Before this commit: robot drok3_description2, 31 links, 30 joints
Links:
- removed link base_footprint_link
Joints:
- removed joint base_link_joint
